File: elec/guider-shield/guider-shield.sch (EAGLE design)
At the start: 18 parts, among them U2 OPENMV3

Commit message: guide-shield almost done
Parts:
- added C4: 0.1uF, sfe:CAP0603-CAP
- added R10, R7, R8, R9: 220R, sfe:RESISTOR0603-RES
- added R5, R6: 4K7, sfe:RESISTOR0603-RES
- added U3: TLP291, guider-shield:TLP283-4-SO016
- added X1: OPENMV3, openmv:OPENMV3
- added X2: MTJ-663X1, guider-shield:ST-4-MTJ-663X1
- U2: value OPENMV3 -> PCA9536-SO8; device openmv:OPENMV3 -> guider-shield:PCA9536-SO8
- renumbered U$3 to U1
Connections:
- new net EAST: U3A.COL, X2.+RA
- new net N$16: R8.1, U3B.C
- new net N$20: R9.1, U3C.C
- new net N$21: R10.1, U3D.C
- new net N$22: R9.2, U2.IO1
- new net N$23: R10.2, U2.IO0
- new net N$24: U3A.EMIT, U3B.EMIT, U3C.EMIT, U3D.EMIT, X2.GND
- new net N$8: R7.1, U3A.C
- new net NORTH: U3B.COL, X2.+DEC
- new net SCL: R5.1, U2.SCL, X1.TXD/SCL
- new net SDA: R6.1, U2.SDA, X1.RXD/SDA
- new net SOUTH: U3C.COL, X2.-DEC
- new net WEST: U3D.COL, X2.-RA
- net 3V3: now also C4.1, R5.2, R6.2, U2.VDD, U3A.A, U3B.A, U3C.A, U3D.A, X1.3.3V; no longer U2.3.3V
- net CHIP_EN: now also X1.ADC/DAC; no longer U2.ADC/DAC
- net GND: now also C4.2, X1.GND
- net IRQ: now also X1.PWM2; no longer U2.PWM2
- net MISO: now also X1.MISO; no longer U2.MISO
- net MOSI: now also X1.MOSI; no longer U2.MOSI
- net N$1: now also R7.2, U2.IO3; no longer U2.TXD/SCL
- net N$2: now also R8.2, U2.IO2; no longer U2.RXD/SDA
- net RESET: now also X1.PWM1; no longer U2.PWM1
- net SCLK: now also X1.SCLK; no longer U2.SCLK
- net SSEL: now also X1.SSEL; no longer U2.SSEL
- net VIN: now also X1.VIN; no longer U2.VIN
Other:
- note added: "additional components here for auto-guider project by Frank Zhao"
