File: elec/guider-shield/v2/guider-shield.brd (EAGLE design)
At the start: 35.6 x 27.9 mm, 11 parts, among them U2 PCA9536-SO8, U3 TLP291, X1 OPENMV3, X2 MTJ-663X1

Commit message: updated guider-shield PCB design
Parts:
- added U$1, U$2: FIDUCIAL, adafruit:FIDUCIAL_1MM
- added U$3: (no value), guider-shield:LOGO
- moved R6 31.6 mm to (22.6, 32.9), turned to 90 degrees
- moved R5 29.8 mm to (24.5, 32.9), turned to 90 degrees
- moved C4 29.2 mm to (15.0, 32.9), turned to 270 degrees
- moved U2 26.2 mm to (18.7, 32.9), turned to 0 degrees
- moved R10 18.2 mm to (15.5, 26.9), turned to 90 degrees
- moved R9 15.1 mm to (18.0, 26.9), turned to 90 degrees
- moved R8 13.1 mm to (20.6, 26.9), turned to 90 degrees
- moved R7 12.5 mm to (23.1, 26.9), turned to 90 degrees
- moved U3 5.36 mm to (19.9, 21.6)
- moved X2 5.33 mm to (17.8, 6.48)
Routing:
- net N$21: track 31.1 -> 1.68 mm
- net SDA: track 13.9 -> 40.5 mm, vias 1 -> 2
- net N$20: track 25.8 -> 1.68 mm
- net SCL: track 14.3 -> 35.5 mm, vias 1 -> 2
- net N$16: track 20.3 -> 1.68 mm
- net N$8: track 14.9 -> 1.68 mm
- net 3V3: track 59.2 -> 67.4 mm, vias 5 -> 4
- net N$22: track 3.30 -> 2.50 mm
- net N$2: track 3.66 -> 3.10 mm
- net EAST: track 3.07 -> 3.58 mm
- net WEST: track 6.88 -> 7.38 mm
- net NORTH: track 6.20 -> 6.71 mm
- net N$24: track 19.4 -> 19.9 mm
Other:
- board size 35.6 x 27.9 mm -> 35.6 x 38.1 mm
