File: elec/guider-shield/v2/guider-shield.sch (EAGLE design)
At the start: 11 parts, among them U2 PCA9536-SO8, U3 TLP291, X1 OPENMV3, X2 MTJ-663X1

Commit message: updated guider-shield PCB design
Parts:
- added U$1, U$2: FIDUCIAL, adafruit:FIDUCIAL
Changed lines of the file:
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@@
 <part name="P+1" library="iofault" deviceset="VIN" device=""/>
 <part name="GND1" library="supply1" deviceset="GND" device=""/>
+<part name="U$1" library="adafruit" deviceset="FIDUCIAL" device=""/>
+<part name="U$2" library="adafruit" deviceset="FIDUCIAL" device=""/>
 <part name="3V2" library="supply" deviceset="3V3" device=""/>
 <part name="U3" library="guider-shield" deviceset="TLP283-4" device="-SO016" value="TLP291"/>
@@
 <instance part="P+1" gate="G$1" x="218.44" y="127"/>
 <instance part="GND1" gate="1" x="226.06" y="78.74"/>
+<instance part="U$1" gate="G$1" x="218.44" y="30.48"/>
+<instance part="U$2" gate="G$1" x="226.06" y="30.48"/>
 <instance part="3V2" gate="G$1" x="226.06" y="137.16"/>
 <instance part="U3" gate="A" x="144.78" y="205.74"/>
